File: Hardware/kompetterx/kompetterx.kicad_sch (KiCad schematic)
At the start: 50 parts, among them J1 OLED_01x04, J2 SPI2_01x05, J3 Programming, J4 +12V PWR, J5 USB_C_Receptacle_USB2.0, Q1 AO3401A, SW1 SW_SPDT, U1 MP2359DJ-LF-Z, U2 STM32F405RGT6, U3 USBLC6-2SC6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

Commit message: Update USB-bug hardware + software
Parts:
- removed J4: +12V PWR, Connector_PinHeader_2.54mm:PinHeader_1x02_P2.54mm_Vertical, symbol New Business Card-rescue:Conn_01x02_Male-Connector
- removed Q1: AO3401A, Package_TO_SOT_SMD:SOT-23, symbol Transistor_FET:AO3401A
- J3: footprint Connector_PinSocket_1.27mm:PinSocket_2x05_P1.27mm_Vertical -> Connector_PinSocket_2.54mm:PinSocket_2x05_P2.54mm_Vertical
Connections:
- net USB_CONN_D+: now also J5.A6 (D+), J5.B6 (D+); no longer J5.A7 (D-), J5.B7 (D-)
- net USB_CONN_D-: now also J5.A7 (D-), J5.B7 (D-); no longer J5.A6 (D+), J5.B6 (D+)
